File: 0008_Buzzer_Module_Classic.kicad_sch (KiCad schematic)
At the start: 13 parts, among them Q1 SS8050-G, SW1 SW_MEC_5E, U1 Buzzer

Commit message: Add files via upload
Parts:
- added D2: LED, LED_SMD:LED_0805_2012Metric, symbol Device:LED
- added R7: 470r, Resistor_SMD:R_0805_2012Metric, symbol Device:R
- added U2: ~, Moduler_:pin_header, symbol moduler_pin:air
- C1, C4: footprint (none) -> Capacitor_SMD:C_0805_2012Metric
- Q1: footprint SOT95P240X115-3N -> Package_TO_SOT_SMD:TSOT-23
- R1, R2, R3: footprint (none) -> Resistor_SMD:R_0805_2012Metric
- SW1: footprint button:button01 -> oled_button:TS046665BK160SMT
- U1: footprint (none) -> Buzzer_Beeper:Buzzer_12x9.5RM7.6
Connections:
- net VCC is gone; now on net +5V: R3.1, R3.1
- net +5V: now also R7.1, U2.7
- net DIN: now also U2.12
- net GND: now also D2.1 (K), U2.9
- net GPIO_01: now also U2.13
- net GPIO_02: now also U2.14
- net SIG: now also U2.15
- new net: D2.2 (A), R7.2
- no-connect marks 1 -> 13
Other:
- note added: "AIR PIN"
- note added: "SENSOR"
- moved on the sheet: C1, C4, D1, Q1, R1, R2, R3, SW1, U1
